File: Horticulture-sensor/HorticultureSensor.kicad_pcb (KiCad board)
At the start: 2 copper layers, 46.9 x 34.8 mm, 24 parts, among them J1 Conn_01x04, J2 Conn_02x05_Odd_Even, J3 Conn_01x03, J4 Conn_01x04, J5 Conn_01x03, J6 Conn_01x02, J7 Conn_01x02, J8 Conn_01x02, Q1 IRLML2030TRPBF, Q2 IRLML2030TRPBF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

Commit message: Resolves #4 #6 #5
Parts:
- removed C2: 1 uF, Capacitor_SMD:C_0805_2012Metric
- removed J7, J8: Conn_01x02, Connector_JST:JST_XH_B2B-XH-AM_1x02_P2.50mm_Vertical
- removed JP1: SolderJumper_2_Open, Jumper:SolderJumper-2_P1.3mm_Open_RoundedPad1.0x1.5mm
- removed Q1, Q2: IRLML2030TRPBF, Package_TO_SOT_SMD:SOT-23
- removed R2: 10 kohm, Resistor_SMD:R_0805_2012Metric
- removed U2: ENS210, Package_DFN_QFN:AMS_QFN-4-1EP_2x2mm_P0.95mm_EP0.7x1.6mm
- removed U3: MCP1700-3302E_TO, Package_TO_SOT_SMD:SOT-23
- C1: value 1 uF -> C_Small
- J1, J4: footprint Connector_JST:JST_XH_S4B-XH-A-1_1x04_P2.50mm_Horizontal -> Connector_Molex:Molex_PicoBlade_53398-0471_1x04-1MP_P1.25mm_Vertical
- J2: moved to B.Cu
- J3, J5: footprint Connector_JST:JST_XH_B3B-XH-A_1x03_P2.50mm_Vertical -> Connector_Molex:Molex_PicoBlade_53398-0371_1x03-1MP_P1.25mm_Vertical
- J6: value Conn_01x02 -> Conn_01x04; footprint Connector_JST:JST_XH_B2B-XH-AM_1x02_P2.50mm_Vertical -> Connector_Molex:Molex_PicoBlade_53398-0471_1x04-1MP_P1.25mm_Vertical; moved to B.Cu
- R1: value 10 kohm -> R_Small
- moved J6 39.4 mm to (150.6, 129.0), turned to 90 degrees
- moved R1 23.3 mm to (162.6, 133.9), turned to 90 degrees
- moved C1 21.6 mm to (162.8, 129.5)
- moved J2 8.63 mm to (162.6, 125.2)
- moved J5 8.40 mm to (166.1, 124.7), turned to 90 degrees
- moved J3 7.23 mm to (166.1, 135.4), turned to 90 degrees
- moved J1 4.68 mm to (157.7, 119.6)
- moved J4 4.07 mm to (157.5, 141.0)
- moved H1 2.85 mm to (148.1, 118.9)
Connections:
- C1 pad 1: VCC -> +3V3
- C1 pad 2: 12V- -> GND
- H1 pad 1: 12V- -> GND
- H2 pad 1: 12V- -> GND
- J1 pad 4: 12V- -> GND
- J2 pad 3: 12V- -> GND
- J2 pad 5: 12V- -> GND
- J3 pad 3: 12V- -> GND
- J4 pad 4: 12V- -> GND
- J5 pad 3: 12V- -> GND
- J6 pad 1: 12V+ -> VCC
- J6 pad 2: control_0 -> UART-tx
- JP2 pad 2: 12V- -> GND
- JP3 pad 2: 12V- -> GND
- JP4 pad 2: 12V- -> GND
- JP5 pad 2: 12V- -> GND
- R1 pad 1: mosfet0 -> +3V3
- R1 pad 2: 12V- -> nRESET
- U1 pad 1: (no net) -> GND
- U1 pad 15: 12V- -> GND
- U1 pad 8: mosfet1 -> UART-tx
- U1 pad 9: mosfet0 -> UART-rx
Routing:
- net 12V-: track 84.8 -> 0.00 mm, vias 4 -> 0
- net I2c-SCL: track 72.1 -> 0.00 mm
- net I2c-SDA: track 66.8 -> 0.00 mm, vias 1 -> 0
- net +3V3: track 63.1 -> 10.3 mm, vias 2 -> 0
- net VCC: track 51.8 -> 0.00 mm
- net mosfet1: track 40.6 -> 0.00 mm, vias 2 -> 0
- net 12V+: track 39.6 -> 0.00 mm
- net GND: track 0.00 -> 29.9 mm, vias 0 -> 2
- net mosfet0: track 29.0 -> 0.00 mm, vias 2 -> 0
- net SWD-SWIO: track 24.3 -> 0.00 mm
- net AnalogSignal0: track 22.5 -> 0.00 mm, vias 2 -> 0
- net SWD-SWCLK: track 22.2 -> 0.00 mm
- net AnalogSignal1: track 20.9 -> 0.00 mm, vias 2 -> 0
- net nRESET: track 17.8 -> 5.45 mm
- net i2c-addr_0: track 11.0 -> 0.00 mm
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- added copper zone on F.Cu, net GND
- removed copper zone on F.Cu, net 12V-
